File: nt-660/nt660.kicad_pcb (KiCad board)
At the start: 2 copper layers, 312 x 96.1 mm, 175 parts, among them J1 USB_mini_micro_B, J2 ISP, K1 KEYSW, K10 KEYSW, K11 KEYSW, K12 KEYSW, K13 KEYSW, K14 KEYSW, K15 KEYSW, K16 KEYSW, K17 KEYSW, K18 KEYSW, K19 KEYSW, K2 KEYSW, K20 KEYSW, K21 KEYSW, K22 KEYSW, K23 KEYSW, K24 KEYSW, K25 KEYSW, K26 KEYSW, K27 KEYSW, K28 KEYSW, K29 KEYSW, K3 KEYSW, K30 KEYSW, K31 KEYSW, K32 KEYSW, K33 KEYSW, K34 KEYSW, K35 KEYSW, K36 KEYSW, K37 KEYSW, K38 KEYSW, K39 KEYSW, K4 KEYSW, K40 KEYSW, K41 KEYSW, K42 KEYSW, K43 KEYSW, K44 KEYSW, K44-1 KEYSW, K46 KEYSW, K46-1 KEYSW, K47 KEYSW, K48 KEYSW, K49 KEYSW, K5 KEYSW, K50 KEYSW, K51 KEYSW, K52 KEYSW, K53 KEYSW, K54 KEYSW, K55 KEYSW, K56 KEYSW, K57 KEYSW, K58 KEYSW, K59 KEYSW, K6 KEYSW, K61 KEYSW, K62 KEYSW, K63 KEYSW, K67 KEYSW, K7 KEYSW, K70 KEYSW, K71 KEYSW, K72 KEYSW, K73 KEYSW, K74 KEYSW, K75 KEYSW, K8 KEYSW, K9 KEYSW, SW1 Reset, U1 ATmega32U4, U2 USBLC6-2SC6, X1 CSTNE16M0V530000R0

Commit message: nt-660 rev1.1
Parts:
- added K62-1: KEYSW, Keeb_switches:CHERRY_PLATE_125H, F.Cu at (35.6, 85.5)
- added K63-1: KEYSW, Keeb_switches:CHERRY_PLATE_125H, F.Cu at (59.4, 85.5)
- added K67-1: KEYSW, Keeb_switches:CHERRY_PCB_600C_H_F, F.Cu at (128.3, 85.5)
- moved D67 15.4 mm to (118.2, 87.3)
- moved D63 4.75 mm to (67.1, 87.3)
- moved D62 2.38 mm to (43.4, 87.3)
Routing:
- net Net-(D67-Pad2): track 8.03 -> 15.8 mm
- net col2: track 386.4 -> 391.2 mm
- net Net-(D63-Pad2): track 8.03 -> 12.6 mm
- net col6: track 277.6 -> 280.0 mm
- net col1: track 467.7 -> 470.1 mm
- net row4: track 313.9 -> 311.5 mm
- net Net-(D62-Pad2): track 8.03 -> 10.2 mm
Other:
- board text added: "rev1.1"
- board text removed: "rev1.0"

Commit message: Update PCB footprints/gerbers
Routing:
- net col1: track 470.1 -> 408.3 mm
- net col0: track 426.5 -> 421.1 mm
- net col2: track 391.2 -> 386.9 mm
- net col5: track 316.8 -> 320.5 mm
- net col3: track 344.6 -> 342.6 mm
- net col4: track 338.5 -> 337.1 mm
- net RST: track 371.3 -> 372.5 mm
- net SCK: track 253.6 -> 252.7 mm
- net VCC: track 491.4 -> 490.7 mm
- net col6: track 280.0 -> 279.4 mm
- net col10: track 183.1 -> 183.6 mm
