File: nt-750/nt750.kicad_pcb (KiCad board)
At the start: 2 copper layers, 347.9 x 123.2 mm, 228 parts, among them J1 S5B-PH-K-S, J2 ISP, K1 KEYSW, K10 KEYSW, K100 KEYSW, K101 KEYSW, K102 KEYSW, K11 KEYSW, K12 KEYSW, K13 KEYSW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

Commit message: Update PCB footprints/gerbers
Routing:
- net col13: track 199.7 -> 196.6 mm
- net col10: track 247.5 -> 246.2 mm
- net col8: track 258.8 -> 258.0 mm
- net GND: vias 8 -> 9
